Commit message: urdf

File: ros2_ws/src/quadruped_description/quadruped/robot.urdf (robot description, URDF)
Before this commit: robot amtq_v2, 13 links, 12 joints
Links:
- added link world
Joints:
- added joint fixed_to_world: type fixed, parent world, child base_link, origin xyz=0 0 0.5 rpy=0 0 0

Commit message: PID 1.0

File: ros2_ws/src/quadruped_description/quadruped/robot.urdf (robot description, URDF)
Before this commit: robot amtq_v2, 14 links, 13 joints
Links:
- removed link world
Joints:
- removed joint fixed_to_world
- joint back_left_coxa_joint: limit lower=-0.954085 upper=1.40211 effort=10 velocity=10 -> lower=-1.5708 upper=1.5708 effort=10 velocity=10
- joint back_left_femur_joint: limit lower=-0 upper=0.785398 effort=10 velocity=10 -> lower=-1.5708 upper=1.5708 effort=10 velocity=10
- joint back_left_tibia_joint: limit lower=-0.783653 upper=0 effort=10 velocity=10 -> lower=-1.5708 upper=1.5708 effort=10 velocity=10
- joint back_right_coxa_joint: limit lower=-1.74824 upper=0.607954 effort=10 velocity=10 -> lower=-1.5708 upper=1.5708 effort=10 velocity=10
- joint back_right_femur_joint: limit lower=-0.162163 upper=0.623235 effort=10 velocity=10 -> lower=-1.5708 upper=1.5708 effort=10 velocity=10
- joint front_left_coxa_joint: limit lower=-1.76112 upper=0.595073 effort=10 velocity=10 -> lower=-1.5708 upper=1.5708 effort=10 velocity=10
- joint front_left_femur_joint: limit lower=0 upper=0.785398 effort=10 velocity=10 -> lower=-1.5708 upper=1.5708 effort=10 velocity=10
- joint front_left_tibia_joint: limit lower=-0.783653 upper=0 effort=10 velocity=10 -> lower=-1.5708 upper=1.5708 effort=10 velocity=10
- joint front_right_coxa_joint: limit lower=-0.53088 upper=1.99985 effort=10 velocity=10 -> lower=-1.5708 upper=1.5708 effort=10 velocity=10
- joint front_right_femur_joint: limit lower=-0 upper=0.785398 effort=10 velocity=10 -> lower=-1.5708 upper=1.5708 effort=10 velocity=10
- joint front_right_tibia_joint: limit lower=-0.774465 upper=0.00918831 effort=10 velocity=10 -> lower=-1.5708 upper=1.5708 effort=10 velocity=10
